File: hardware/breathy/breathy.kicad_pcb (KiCad board)
At the start: 2 copper layers, 15 parts, among them J2 USB_C_Receptacle_USB2.0_16P, Q1 MMBT3906, Q2 2SAR572D3TL1, Q3 PMV37ENEAR, Q4 PMV37ENEAR, U1 AZ431AN, U2 ESP32-C3-MINI-1, U3 USBLC6-2SC6, U4 TLV9002IDDFR, U5 DW01A, U6 TLV9002, U7 AZ431AN

Commit message: adding pdf schematics
Parts:
- added C1: 0.1u, Capacitor_SMD:C_0805_2012Metric, F.Cu at (187.2, 65.8)
- added C10: 1nF, Capacitor_SMD:C_0805_2012Metric, F.Cu at (172.2, 36.6)
- added C11: 1nF, Capacitor_SMD:C_0805_2012Metric, F.Cu at (172.2, 39.6)
- added C12: 1nF, Capacitor_SMD:C_0805_2012Metric, F.Cu at (172.2, 42.6)
- added C13: 1u, Capacitor_SMD:C_1206_3216Metric, F.Cu at (173.3, 48.6)
- added C14: 0.1u, Capacitor_SMD:C_0805_2012Metric, F.Cu at (238.6, 75.6)
- added C15: 0.1u, Capacitor_SMD:C_0805_2012Metric, F.Cu at (103.8, 109.4)
- added C2: 10u, Capacitor_SMD:C_1206_3216Metric, F.Cu at (187.1, 68.4)
- added C3: 10u, Capacitor_SMD:C_1206_3216Metric, F.Cu at (187.1, 71.6)
- added C4: 0.1u, Capacitor_SMD:C_0805_2012Metric, F.Cu at (140.3, 122.4)
- added C5: 0.1u, Capacitor_SMD:C_0805_2012Metric, F.Cu at (145.8, 121.2)
- added C6: 0.1u, Capacitor_SMD:C_0805_2012Metric, F.Cu at (83.1, 80.1)
- added C7: 1u, Capacitor_SMD:C_1206_3216Metric, F.Cu at (103.5, 75.2)
- added C8: 0.1u, Capacitor_SMD:C_0805_2012Metric, F.Cu at (172.0, 26.8)
- added C9: 0.1u, Capacitor_SMD:C_0805_2012Metric, F.Cu at (173.6, 32.0)
- added D1: LED R, LED_SMD:LED_1206_3216Metric, F.Cu at (161.8, 91.4)
- added D2: D_Schottky, Diode_SMD:D_SOD-323_HandSoldering, F.Cu at (197.6, 41.2)
- added D3: D_Schottky, Diode_SMD:D_SOD-323_HandSoldering, F.Cu at (197.6, 44.1)
- added D4: LED G, LED_SMD:LED_1206_3216Metric, F.Cu at (179.0, 48.6)
- added F1: Polyfuse, Capacitor_SMD:C_1206_3216Metric, F.Cu at (165.4, 85.9)
- added J1: Conn_01x04_Pin, Connector_PinHeader_2.54mm:PinHeader_1x04_P2.54mm_Vertical, F.Cu at (184.5, 91.0)
- added J2: Supply sel, Connector_PinHeader_2.54mm:PinHeader_1x03_P2.54mm_Vertical, F.Cu at (151.4, 121.9)
- added J3: EPD, Connector_PinHeader_2.54mm:PinHeader_1x08_P2.54mm_Horizontal, F.Cu at (70.2, 33.3)
- added J5: Conn_01x02_Pin, Connector_PinHeader_2.54mm:PinHeader_1x02_P2.54mm_Vertical, F.Cu at (209.1, 41.6)
- added J6: Screw_Terminal_01x02, TerminalBlock:TerminalBlock_MaiXu_MX126-5.0-02P_1x02_P5.00mm, F.Cu at (241.8, 87.6)
- added JP1: JMP, Jumper:SolderJumper-2_P1.3mm_Open_TrianglePad1.0x1.5mm, F.Cu at (156.2, 126.2)
- added JP2: Jumper_2_Small_Open, Jumper:SolderJumper-2_P1.3mm_Open_TrianglePad1.0x1.5mm, F.Cu at (214.6, 43.0)
- added Q1: SL2301S, Package_TO_SOT_SMD:SOT-23, F.Cu at (69.1, 27.6)
- added Q2: MMBT3906, Package_TO_SOT_SMD:SOT-23, F.Cu at (193.9, 30.0)
- added Q5: PMV37ENEAR, PMV37ENEAR:SOT95P230X110-3N, F.Cu at (161.7, 47.6)
- added Q6: PMV37ENEAR, PMV37ENEAR:SOT95P230X110-3N, F.Cu at (161.7, 51.8)
- added R10: 5.1k, Resistor_SMD:R_0805_2012Metric, F.Cu at (173.1, 79.4)
- added R11: 150, Resistor_SMD:R_0805_2012Metric, F.Cu at (161.8, 95.9)
- added R12: 100k, Resistor_SMD:R_1206_3216Metric, F.Cu at (34.3, 180.8)
- added R13: 100k, Resistor_SMD:R_1206_3216Metric, F.Cu at (167.3, 37.1)
- added R14: 100k, Resistor_SMD:R_1206_3216Metric, F.Cu at (167.3, 40.4)
- added R15: 1k, Resistor_SMD:R_1206_3216Metric, F.Cu at (167.3, 43.7)
- added R16: 0R100, Resistor_SMD:R_2010_5025Metric_Pad1.40x2.65mm_HandSolder, F.Cu at (204.9, 26.4)
- added R17: 10k, Resistor_SMD:R_0805_2012Metric, F.Cu at (200.5, 31.2)
- added R18: 10k, Resistor_SMD:R_0805_2012Metric, F.Cu at (200.5, 34.1)
- added R19: 5.1k, Resistor_SMD:R_0805_2012Metric, F.Cu at (200.5, 37.1)
- added R2: 5.1k, Resistor_SMD:R_0805_2012Metric, F.Cu at (109.1, 113.8)
- added R20: 10k, Resistor_SMD:R_0805_2012Metric, F.Cu at (152.5, 38.0)
- added R21: 10k, Resistor_SMD:R_0805_2012Metric, F.Cu at (194.7, 36.5)
- added R22: 150, Resistor_SMD:R_0805_2012Metric, F.Cu at (161.5, 37.8)
- added R23: 0R, Resistor_SMD:R_0805_2012Metric, F.Cu at (161.5, 40.4)
- added R24: 1k, Resistor_SMD:R_1206_3216Metric, F.Cu at (167.3, 47.0)
- added R25: 10k, Resistor_SMD:R_0805_2012Metric, F.Cu at (161.5, 43.3)
- added R26: 6k8, Resistor_SMD:R_0805_2012Metric, F.Cu at (156.9, 38.0)
- added R27: 10k, Resistor_SMD:R_0805_2012Metric, F.Cu at (156.9, 41.0)
- added R28: 100k, Resistor_SMD:R_1206_3216Metric, F.Cu at (167.3, 50.3)
- added R3: 10k, Resistor_SMD:R_0805_2012Metric, F.Cu at (82.7, 71.8)
- added R4: 10k, Resistor_SMD:R_0805_2012Metric, F.Cu at (103.3, 66.4)
- added R5: 10k, Resistor_SMD:R_0805_2012Metric, F.Cu at (109.5, 79.0)
- added R6: 10k, Resistor_SMD:R_0805_2012Metric, F.Cu at (165.9, 81.4)
- added R7: 5.1k, Resistor_SMD:R_0805_2012Metric, F.Cu at (178.3, 93.2)
- added R8: 5.1k, Resistor_SMD:R_0805_2012Metric, F.Cu at (178.3, 96.6)
- added R9: 10k, Resistor_SMD:R_0805_2012Metric, F.Cu at (169.7, 81.4)
- added RV1: 20K, Potentiometer_SMD:Potentiometer_Bourns_TC33X_Vertical, F.Cu at (159.8, 27.6)
- added RV2: 20K, Potentiometer_SMD:Potentiometer_Bourns_TC33X_Vertical, F.Cu at (159.8, 32.4)
- added SW1: SW_Push, Button_Switch_SMD:SW_Push_1P1T_NO_CK_KSC9xxG, F.Cu at (112.7, 70.4)
- added SW2: SW_Push, Jumper:SolderJumper-2_P1.3mm_Open_TrianglePad1.0x1.5mm, F.Cu at (103.1, 71.0)
- added SW3: CHG RST, Button_Switch_SMD:SW_Push_1P1T_NO_CK_KSC9xxG, F.Cu at (151.7, 48.6)
- added TP1: TestPoint, TestPoint:TestPoint_Pad_D1.5mm, F.Cu at (140.8, 127.5)
- added TP2: TestPoint, TestPoint:TestPoint_Pad_D1.5mm, F.Cu at (160.4, 87.2)
- added TP3: TestPoint, TestPoint:TestPoint_Pad_D1.5mm, F.Cu at (145.4, 39.2)
- added TP4: TestPoint, TestPoint:TestPoint_Pad_D1.5mm, F.Cu at (145.4, 42.8)
- added U1: XC6503D301MR-G, Package_TO_SOT_SMD:SC-74A-5_1.55x2.9mm_P0.95mm, F.Cu at (145.2, 126.8)
- added U10: BME690, Package_LGA:Bosch_LGA-8_3x3mm_P0.8mm_ClockwisePinNumbering, F.Cu at (104.0, 114.0)
- added U11: DS18B20, Package_TO_SOT_THT:TO-92_Inline, F.Cu at (97.1, 114.6)
- added U3: MAX17048G+, MAX17048:21-0168_T822&plus_3_MXM-M, F.Cu at (83.2, 75.7)
- R1: value 0R100 -> 5.1k; footprint Resistor_SMD:R_2010_5025Metric_Pad1.40x2.65mm_HandSolder -> Resistor_SMD:R_0805_2012Metric
- R29: renamed from R6; footprint Resistor_SMD:R_1206_3216Metric_Pad1.30x1.75mm_HandSolder -> Resistor_SMD:R_0805_2012Metric
- R30: renamed from R7; footprint Resistor_SMD:R_1206_3216Metric_Pad1.30x1.75mm_HandSolder -> Resistor_SMD:R_1206_3216Metric
- U2: value ESP32-C3-MINI-1 -> ESP32-C6-MINI-1/U; footprint PCM_Espressif:ESP32-C3-MINI-1 -> PCM_Espressif:ESP32-C6-MINI-1
- U6: renamed from U4; value TLV9002IDDFR -> TLV9002
- moved R29 119.9 mm to (244.9, 69.2)
- moved Q7 114.3 mm to (238.8, 70.6)
- moved Q8 114.3 mm to (243.8, 76.0)
- moved Q3 111.9 mm to (212.1, 34.1)
- moved U9 110.9 mm to (250.2, 72.8)
- moved Q4 100.1 mm to (203.6, 41.8)
- moved R30 99.7 mm to (245.1, 71.8)
- moved U5 91.2 mm to (166.3, 32.7)
- moved U6 91.2 mm to (166.3, 28.1)
- moved U7 82.6 mm to (148.2, 30.8)
- moved U8 82.6 mm to (153.6, 28.3)
- moved U4 50.2 mm to (170.4, 85.8), turned to -90 degrees
- moved U2 47.9 mm to (187.1, 80.4), turned to -90 degrees
- moved R1 44.0 mm to (109.1, 110.8)
- moved J4 11.2 mm to (170.5, 94.2)
- renumbered J2 to J4, Q2 to Q3, Q1 to Q4, Q3 to Q7, Q4 to Q8, U3 to U4, U6 to U5, U1 to U8, U5 to U9
Connections:
- Q3 pad 1: unconnected-(Q2-B-Pad1) -> Net-(Q3-B)
- Q3 pad 2: unconnected-(Q2-C-Pad2) -> Net-(J5-Pin_2)
- Q3 pad 3: unconnected-(Q2-E-Pad3) -> /Charger/V_shunt
- Q4 pad 1: unconnected-(Q1-B-Pad1) -> Net-(D2-K)
- Q4 pad 2: unconnected-(Q1-E-Pad2) -> Net-(Q3-B)
- Q4 pad 3: unconnected-(Q1-C-Pad3) -> GND
- R1 pad 1: unconnected-(R1-Pad1) -> /i2c_scl
- R1 pad 2: unconnected-(R1-Pad2) -> +3V0
- U2 pad 12: unconnected-(U2-GPIO0/ADC1_CH0/XTAL_32K_P-Pad12) -> /usb_conn
- U2 pad 13: unconnected-(U2-GPIO1/ADC1_CH1/XTAL_32K_N-Pad13) -> /chrg_end_n
- U2 pad 15: unconnected-(U2-NC-Pad15) -> /i2c_sda
- U2 pad 16: unconnected-(U2-GPIO10-Pad16) -> /i2c_scl
- U2 pad 17: unconnected-(U2-NC-Pad17) -> /D-
- U2 pad 18: unconnected-(U2-GPIO4/ADC1_CH4-Pad18) -> /D+
- U2 pad 19: unconnected-(U2-GPIO5/ADC2_CH0-Pad19) -> /1w
- U2 pad 20: unconnected-(U2-GPIO6-Pad20) -> /SDA
- U2 pad 22: unconnected-(U2-GPIO8-Pad22) -> /gpio8_pu
- U2 pad 23: unconnected-(U2-GPIO9-Pad23) -> /gpio9_dl
- U2 pad 24: unconnected-(U2-NC-Pad24) -> /SCL
- U2 pad 25: unconnected-(U2-NC-Pad25) -> /CS
- U2 pad 26: /D- -> /D/C
- U2 pad 27: /D+ -> /RES
- U2 pad 28: unconnected-(U2-NC-Pad28) -> /BUSY
- U2 pad 3: unconnected-(U2-3V3-Pad3) -> +3V0
- U2 pad 30: unconnected-(U2-GPIO20/U0RXD-Pad30) -> Net-(J1-Pin_2)
- U2 pad 31: unconnected-(U2-GPIO21/U0TXD-Pad31) -> Net-(J1-Pin_3)
- U2 pad 5: unconnected-(U2-GPIO2/ADC1_CH2-Pad5) -> /batt_alrt
- U2 pad 8: unconnected-(U2-EN/CHIP_PU-Pad8) -> /chip_en
- U5 pad 1: unconnected-(U6-Pad1) -> Net-(U5A--)
- U5 pad 2: unconnected-(U6A---Pad2) -> Net-(U5A--)
- U5 pad 3: unconnected-(U6A-+-Pad3) -> /Charger/i_max
- U5 pad 5: unconnected-(U6B-+-Pad5) -> /Charger/i_max
- U5 pad 6: unconnected-(U6B---Pad6) -> Net-(U5B--)
- U5 pad 7: unconnected-(U6-Pad7) -> Net-(D2-A)
- U6 pad 1: unconnected-(U4-Pad1) -> Net-(D3-A)
- U6 pad 2: unconnected-(U4A---Pad2) -> Net-(U6A--)
- U6 pad 3: unconnected-(U4A-+-Pad3) -> Net-(U6A-+)
- U6 pad 5: unconnected-(U4B-+-Pad5) -> /Charger/i_end
- U6 pad 6: unconnected-(U4B---Pad6) -> /Charger/V_shunt
- U6 pad 7: unconnected-(U4-Pad7) -> Net-(Q6-Pad2)
- U7 pad 1: unconnected-(U7-REF-Pad1) -> VBUS
- U7 pad 2: unconnected-(U7-K-Pad2) -> VBUS
- U7 pad 3: unconnected-(U7-A-Pad3) -> Net-(U7-A)
- U8 pad 1: unconnected-(U1-REF-Pad1) -> Net-(U8-REF)
- U8 pad 2: unconnected-(U1-K-Pad2) -> Net-(U8-K)
- U8 pad 3: unconnected-(U1-A-Pad3) -> GND
Routing:
- net /D-: track 0.00 -> 22.0 mm, vias 0 -> 2
- net /D+: track 0.00 -> 18.5 mm
- net VBUS: track 0.00 -> 16.5 mm, vias 0 -> 2
- net /usb_conn: track 0.00 -> 15.5 mm
- net Net-(F1-Pad1): track 0.00 -> 13.1 mm, vias 0 -> 2
- net Net-(J4-CC1): track 0.00 -> 11.5 mm
- net Net-(J4-CC2): track 0.00 -> 6.80 mm
- net Net-(R10-Pad2): track 0.00 -> 2.65 mm
- net Net-(D1-K): track 0.00 -> 2.20 mm
