File: hardware/breathy/breathy.kicad_sch (KiCad schematic)
At the start: 24 parts, among them J1 Conn_01x04_Pin, J2 USB_C_Receptacle_USB2.0_16P, J4 EPD, Q6 SL2301S, SW2 SW_Push, SW3 SW_Push, U2 XC6503D301MR-G, U3 USBLC6-2SC6, U8 ESP32-C6-MINI-1/U

Commit message: test points, headers, indicators, no battery sim
Parts:
- added C14: 10u, symbol Device:C_Small
- added C15: 0.1u, symbol Device:C_Small
- added D4: LED R, LED_SMD:LED_1206_3216Metric, symbol Device:LED
- added J5: Supply sel, symbol Connector:Conn_01x03_Pin
- added JP1: JMP, Jumper:SolderJumper-2_P1.3mm_Open_TrianglePad1.0x1.5mm, symbol Jumper:Jumper_2_Small_Open
- added R30: 10k, symbol Device:R_Small
- added R31: 150, symbol Device:R_Small
- added TP3, TP4: TestPoint, symbol Connector:TestPoint
- added U12: MAX17048G+, 21-0168_T822+3_MXM, symbol MAX17048:MAX17048G+
- C10: now fitted
- C8: value 22u -> 10u
Connections:
- net +3V0: now also C14.1, R30.2, TP4.1
- net +BATT: now also C15.1, J5.3 (Pin_3), JP1.1 (A), U12.2 (CELL), U12.3 (VDD); no longer C11.1, U2.1 (VIN), U2.3 (CE)
- net GND: now also C14.2, C15.2, R31.1, U12.1 (CTG), U12.4 (GND), U12.6 (QSTRT), U12.9 (EPAD)
- net VBUS: now also D4.2 (A), J5.1 (Pin_1), TP3.1
- net batt_alrt: now reaches U8.5 (GPIO2/ADC1_CH2)
- net batt_alrt: now also R30.1, U12.5 (*ALRT)
- net sensors/i2c_scl renamed i2c_scl
- net i2c_scl: now also U12.7 (SCL)
- net sensors/i2c_sda renamed i2c_sda
- net i2c_sda: now also U12.8 (SDA)
- new net: C11.1, J5.2 (Pin_2), JP1.2 (B), U2.1 (VIN), U2.3 (CE)
- new net: D4.1 (K), R31.2
- no-connect marks 8 -> 7
Other:
- sheet battery: file batteery.kicad_sch -> battery.kicad_sch
- sheet sensors: file sensors_display.kicad_sch -> sensors.kicad_sch
- note added: "addr 0x36"
- note added: "test epd true consumption w&w/o LDO"
- moved on the sheet: C11, C12, F1, J2, R24, R25, R26, R27, R28, R4, R5, U2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

Commit message: adding pdf schematics
Parts:
- C1: renamed from C10; footprint (none) -> Capacitor_SMD:C_0805_2012Metric
- C2: renamed from C14; footprint (none) -> Capacitor_SMD:C_1206_3216Metric
- C3: renamed from C8; footprint (none) -> Capacitor_SMD:C_1206_3216Metric
- C4: renamed from C11; footprint (none) -> Capacitor_SMD:C_0805_2012Metric
- C5: renamed from C12; footprint (none) -> Capacitor_SMD:C_0805_2012Metric
- C6: renamed from C15; footprint (none) -> Capacitor_SMD:C_0805_2012Metric
- C7: renamed from C9; footprint (none) -> Capacitor_SMD:C_1206_3216Metric
- F1: footprint (none) -> Capacitor_SMD:C_1206_3216Metric
- J1: footprint (none) -> Connector_PinHeader_2.54mm:PinHeader_1x04_P2.54mm_Vertical
- J2: renamed from J5; footprint (none) -> Connector_PinHeader_2.54mm:PinHeader_1x03_P2.54mm_Vertical
- J3: renamed from J4; footprint (none) -> Connector_PinHeader_2.54mm:PinHeader_1x08_P2.54mm_Horizontal
- R1: renamed from R27; footprint (none) -> Resistor_SMD:R_0805_2012Metric
- R10: renamed from R26; footprint (none) -> Resistor_SMD:R_0805_2012Metric
- R11: renamed from R31; footprint (none) -> Resistor_SMD:R_0805_2012Metric
- R2: renamed from R28; footprint (none) -> Resistor_SMD:R_0805_2012Metric
- R3: renamed from R30; footprint (none) -> Resistor_SMD:R_0805_2012Metric
- R4: renamed from R23; footprint (none) -> Resistor_SMD:R_0805_2012Metric
- R5: renamed from R22; footprint (none) -> Resistor_SMD:R_0805_2012Metric
- R6: renamed from R24; footprint (none) -> Resistor_SMD:R_0805_2012Metric
- R7: renamed from R5; footprint (none) -> Resistor_SMD:R_0805_2012Metric
- R8: renamed from R4; footprint (none) -> Resistor_SMD:R_0805_2012Metric
- R9: renamed from R25; footprint (none) -> Resistor_SMD:R_0805_2012Metric
- TP1: renamed from TP4; footprint (none) -> TestPoint:TestPoint_Pad_D1.5mm
- TP2: renamed from TP3; footprint (none) -> TestPoint:TestPoint_Pad_D1.5mm
- U3: renamed from U12; footprint 21-0168_T822+3_MXM -> MAX17048:21-0168_T822&plus_3_MXM-M
- renumbered D4 to D1, J2 to J4, Q6 to Q1, SW2 to SW1, SW3 to SW2, U2 to U1, U8 to U2, U3 to U4
