File: hardware/breathy/sensors.kicad_sch (KiCad schematic)
At the start: 0 parts

Commit message: test points, headers, indicators, no battery sim
Parts:
- added C13: 0.1u, symbol Device:C_Small
- added U10: DS18B20, Package_TO_SOT_THT:TO-92_Inline, symbol Sensor_Temperature:DS18B20
- added U9: BME690, Package_LGA:Bosch_LGA-8_3x3mm_P0.8mm_ClockwisePinNumbering, symbol Sensor:BME680
Connections:
- new net +3V0: C13.2, U9.2 (CSB), U9.6 (VDDIO), U9.8 (VDD)
- new net 1w: U10.2 (DQ)
- new net 3V_SENS: U10.3 (V_{DD})
- new net GND: C13.1, U10.1 (GND), U9.1 (GND), U9.5 (SDO), U9.7 (GND)
- new net i2c_scl: U9.4 (SCK)
- new net i2c_sda: U9.3 (SDI)
Other:
- note added: "addr 0x76"

Commit message: adding pdf schematics
Parts:
- C15: renamed from C13; footprint (none) -> Capacitor_SMD:C_0805_2012Metric
- renumbered U9 to U10, U10 to U11
Changed lines of the file:
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@@
 		(dnp no)
 		(fields_autoplaced yes)
-		(property "Reference" "#PWR023"
+		(property "Reference" "#PWR032"
 			(at 100.33 113.03 0)
 			(hide yes)
@@
 			(project "breathy"
 				(path "/b1c49805-8a08-4cdd-9984-c6cc27843db8/b22c8a24-e204-45bc-8b3b-514f2bbf507e"
-					(reference "#PWR023")
+					(reference "#PWR032")
 					(unit 1)
 				)
@@
 		(in_pos_files yes)
 		(dnp no)
-		(property "Reference" "U9"
+		(property "Reference" "U10"
 			(at 115.57 52.0699 0)
 			(show_name no)
@@
 			(project "breathy"
 				(path "/b1c49805-8a08-4cdd-9984-c6cc27843db8/b22c8a24-e204-45bc-8b3b-514f2bbf507e"
-					(reference "U9")
+					(reference "U10")
 					(unit 1)
 				)
@@
 		(dnp no)
 		(fields_autoplaced yes)
-		(property "Reference" "#PWR029"
+		(property "Reference" "#PWR030"
 			(at 106.68 26.67 0)
 			(hide yes)
@@
 			(project "breathy"
 				(path "/b1c49805-8a08-4cdd-9984-c6cc27843db8/b22c8a24-e204-45bc-8b3b-514f2bbf507e"
-					(reference "#PWR029")
+					(reference "#PWR030")
 					(unit 1)
 				)
@@
 		(in_pos_files yes)
 		(dnp no)
-		(property "Reference" "U10"
+		(property "Reference" "U11"
 			(at 106.68 97.7899 0)
 			(show_name no)
@@
 			(project "breathy"
 				(path "/b1c49805-8a08-4cdd-9984-c6cc27843db8/b22c8a24-e204-45bc-8b3b-514f2bbf507e"
-					(reference "U10")
+					(reference "U11")
 					(unit 1)
 				)
@@
 		(dnp no)
 		(fields_autoplaced yes)
-		(property "Reference" "#PWR027"
+		(property "Reference" "#PWR029"
 			(at 101.6 36.83 0)
 			(hide yes)
@@
 			(project "breathy"
 				(path "/b1c49805-8a08-4cdd-9984-c6cc27843db8/b22c8a24-e204-45bc-8b3b-514f2bbf507e"
-					(reference "#PWR027")
+					(reference "#PWR029")
 					(unit 1)
 				)
@@
 		(dnp no)
 		(fields_autoplaced yes)
-		(property "Reference" "C13"
+		(property "Reference" "C15"
 			(at 109.22 34.2962 0)
 			(show_name no)
@@
 			)
 		)
-		(property "Footprint" ""
+		(property "Footprint" "Capacitor_SMD:C_0805_2012Metric"
 			(at 106.68 35.56 0)
 			(hide yes)
@@
 			(project "breathy"
 				(path "/b1c49805-8a08-4cdd-9984-c6cc27843db8/b22c8a24-e204-45bc-8b3b-514f2bbf507e"
-					(reference "C13")
+					(reference "C15")
 					(unit 1)
 				)
@@
 		(dnp no)
 		(fields_autoplaced yes)
-		(property "Reference" "#PWR024"
+		(property "Reference" "#PWR031"
 			(at 104.14 76.2 0)
 			(hide yes)
@@
 			(project "breathy"
 				(path "/b1c49805-8a08-4cdd-9984-c6cc27843db8/b22c8a24-e204-45bc-8b3b-514f2bbf507e"
-					(reference "#PWR024")
-					(unit 1)
-				)
+					(reference "#PWR031")
+					(unit 1)
+				)
